File: Relay Module/Relay2.sch (KiCad schematic (older format))
At the start: 19 parts, among them J1 , J2 Conn_01x02, J3Y1 S8050, J3Y2 S8050, K1 SANYOU_SRD_Form_C, K2 SANYOU_SRD_Form_C, U1 PC817

Commit message: Add files via upload
Parts:
- J1: footprint Connector_PinHeader_1.27mm:PinHeader_1x04_P1.27mm_Vertical -> Connector_PinHeader_2.00mm:PinHeader_1x04_P2.00mm_Vertical
- J2, Jumper1: footprint Connector_PinHeader_1.27mm:PinHeader_1x02_P1.27mm_Vertical -> Connector_PinHeader_2.00mm:PinHeader_1x02_P2.00mm_Vertical
Changed lines of the file:
@@
 F 0 "J1" H 3330 4742 50  0000 L CNN
 F 1 " " H 3330 4651 50  0000 L CNN
-F 2 "Connector_PinHeader_1.27mm:PinHeader_1x04_P1.27mm_Vertical" H 3250 4750 50  0001 C CNN
+F 2 "Connector_PinHeader_2.00mm:PinHeader_1x04_P2.00mm_Vertical" H 3250 4750 50  0001 C CNN
 F 3 "~" H 3250 4750 50  0001 C CNN
 	1    3250 4750
@@
 F 0 "J2" V 4372 4380 50  0000 L CNN
 F 1 "Conn_01x02" V 4463 4380 50  0000 L CNN
-F 2 "Connector_PinHeader_1.27mm:PinHeader_1x02_P1.27mm_Vertical" H 4500 4300 50  0001 C CNN
+F 2 "Connector_PinHeader_2.00mm:PinHeader_1x02_P2.00mm_Vertical" H 4500 4300 50  0001 C CNN
 F 3 "~" H 4500 4300 50  0001 C CNN
 	1    4500 4300
@@
 F 0 "Jumper1" V 4372 1830 50  0000 L CNN
 F 1 " " V 4463 1830 50  0000 L CNN
-F 2 "Connector_PinHeader_1.27mm:PinHeader_1x02_P1.27mm_Vertical" H 4500 1750 50  0001 C CNN
+F 2 "Connector_PinHeader_2.00mm:PinHeader_1x02_P2.00mm_Vertical" H 4500 1750 50  0001 C CNN
 F 3 "~" H 4500 1750 50  0001 C CNN
 	1    4500 1750
