File: RelayModule/Relay2.kicad_pcb (KiCad board)
At the start: 2 copper layers, 61 x 36.8 mm, 19 parts, among them J1 , J2 Conn_01x02, J3Y S8050, K1 , K2 

Commit message: Add files via upload
Parts:
- J1: footprint Connector_PinHeader_2.00mm:PinHeader_1x04_P2.00mm_Vertical -> Connector_PinHeader_2.54mm:PinHeader_1x04_P2.54mm_Vertical
- J2, Jumper1: footprint Connector_PinHeader_2.00mm:PinHeader_1x02_P2.00mm_Vertical -> Connector_PinHeader_2.54mm:PinHeader_1x02_P2.54mm_Vertical
Routing:
- net Net-(D3-Pad1): track 11.2 -> 9.51 mm
- net Net-(D1-Pad2): track 19.7 -> 21.0 mm
- net Net-(J1-Pad1): track 62.3 -> 61.8 mm
